Commit message: whill.xacro update

File: vehicle/whill_vehicle_launch/whill_vehicle_description/urdf/whill.xacro (robot description, xacro)
@@ -6,5 +6,5 @@
   <link name="base_link">
     <visual>
-      <origin xyz="${vehicle_info['/**']['ros__parameters']['wheel_base']/2.0} 0 0" rpy="${pi/2.0} 0 ${pi}"/>
+      <origin xyz="0 0 0" rpy="${pi/2.0} 0 ${pi}"/>
       <geometry>
         <mesh filename="package://whill_vehicle_description/mesh/whill.fbx" scale="0.12 0.12 0.12"/>
