Commit message: modify vehicle.xacro

File: vehicle/whill_vehicle_launch/whill_vehicle_description/urdf/vehicle.xacro (robot description, xacro)
@@ -7,5 +7,5 @@
   <xacro:include filename="$(find whill_vehicle_description)/urdf/whill.xacro"/>
   <!-- sensors -->
-  <xacro:property name="sensor_model_property" value="$(arg sensor_model)"/>
-  <xacro:include filename="$(find whill_sensor_kit_description)/urdf/sensors.xacro"/>
+  <!-- <xacro:property name="sensor_model_property" value="$(arg sensor_model)"/>
+  <xacro:include filename="$(find whill_sensor_kit_description)/urdf/sensors.xacro"/> -->
 </robot>
